File: PCB/Datalogger-v2/Datalogger-v2.kicad_sch (KiCad schematic)
At the start: 24 parts, among them U1 Micro SD Card Adapter, U7 TP4056, U8 ESP32 DEV KIT DOIT

Commit message: Update PCB files
- Add Libraries folder.
- Update schematic.
- Update PCB layout.
Parts:
- U8: footprint (none) -> New_Datalogger:DOIT-ESP32-DEVKIT-V1
Connections:
- net 5V/2A: now also U8.1 (3V3)
- net GND: now also U8.2 (GND)
- net at U8.5 (ADC/D4): now also U5.4 (SCL)
- net at U8.6 (UA2RX/D16): now also U5.3 (SDA)
Other:
- moved on the sheet: R1, R2, U8
