File: 02_PCB/Datalogger-v2/Datalogger-v2.kicad_sch (KiCad schematic)
At the start: 26 parts, among them U1 Micro SD Card Adapter, U7 TP4056, U8 ESP32 DEV KIT DOIT

Commit message: Update PCB layout and schematic
- Removed Step-Up Converter and Battery Charger
- Added button
- Fixed errors
Parts:
- removed BT1: Battery_Cell, symbol Device:Battery_Cell
- removed R3: 2kΩ, Resistor_THT:R_Axial_DIN0207_L6.3mm_D2.5mm_P10.16mm_Horizontal, symbol PCM_SL_Resistors:Resistor
- removed R4: 560Ω, Resistor_THT:R_Axial_DIN0207_L6.3mm_D2.5mm_P10.16mm_Horizontal, symbol PCM_SL_Resistors:Resistor
- removed U2: (no value), Datalogger-v2:MT3608, symbol Datalogger-v2:MT3608
- removed U7: TP4056, Datalogger-v2:TP4056, symbol Datalogger-v2:TP4056
- added SW1: SW_Push, Button_Switch_THT:SW_PUSH_6mm, symbol Switch:SW_Push
- R2: value 4.7Ω -> 4.7kΩ
- R8: renamed from R10; value 4.7Ω -> 4.7kΩ
- R9: renamed from R11; value 4.7Ω -> 4.7kΩ
- renumbered R5 to R3, R6 to R4, R7 to R5, R8 to R6, R9 to R7
Connections:
- net +5V: now also U5.4 (5V); no longer U5.2 (VIN)
- net GND: now also SW1.2
- net at R8.1: now also U5.2 (SDA); no longer U5.3 (SDA)
- net at R9.1: now also U5.3 (SCL); no longer U5.4 (SCL)
- net at U8.12 (ADC/D12): now also SW1.1
